Commit message: Added color to gazebo top plate

File: husky_gazebo/urdf/ur5_arm.gazebo.xacro (robot description, xacro)
@@ -22,4 +22,7 @@
 -->
 <robot name="husky_ur5_arm_gazebo" xmlns:xacro="http://ros.org/wiki/xacro">
+  <gazebo reference="ur5_top_plate_link">
+     <material>Gazebo/Black</material>
+  </gazebo>
  <!-- Gazebo references for self collide -->
   <gazebo reference="ur5_arm_shoulder_link">

Commit message: Changed black to dark grey

File: husky_gazebo/urdf/ur5_arm.gazebo.xacro (robot description, xacro)
@@ -23,5 +23,5 @@
 <robot name="husky_ur5_arm_gazebo" xmlns:xacro="http://ros.org/wiki/xacro">
   <gazebo reference="ur5_top_plate_link">
-     <material>Gazebo/Black</material>
+     <material>Gazebo/DarkGrey</material>
   </gazebo>
  <!-- Gazebo references for self collide -->
