Commit message: RP-264 Remove multirobot prefixing, experiment later

File: husky_gazebo/urdf/description.gazebo.xacro (robot description, xacro)
@@ -23,4 +23,4 @@
 <robot name="husky_description" xmlns:xacro="http://ros.org/wiki/xacro">
   <xacro:include filename="$(find husky_gazebo)/urdf/husky.gazebo.xacro" />
-  <xacro:husky_gazebo_robot prefix="" />
+  <xacro:husky_gazebo_robot />
 </robot>

File: husky_gazebo/urdf/husky.gazebo.xacro (robot description, xacro)
@@ -27,6 +27,12 @@
   <xacro:include filename="$(find husky_description)/urdf/husky.urdf.xacro" />
   <xacro:include filename="$(find husky_gazebo)/urdf/sick_lms100.urdf.xacro" />
-  <xacro:macro name="husky_gazebo_robot" params="prefix">
-    <xacro:husky_robot prefix="${prefix}" />
+  <xacro:macro name="husky_gazebo_robot">
+    <xacro:husky_robot />
+    <!-- Gazebo plugin for ROS Control -->
+    <gazebo>
+      <plugin name="gazebo_ros_control" filename="libgazebo_ros_control.so">
+        <robotNamespace>/</robotNamespace>
+      </plugin>
+    </gazebo>
     <xacro:if value="$(arg front_laser)">
       <link name="sick_bracket_link">
@@ -54,9 +60,4 @@
       </joint>
     </xacro:if>
-    <gazebo>
-      <plugin name="gazebo_ros_control" filename="libgazebo_ros_control.so">
-        <robotNamespace>/</robotNamespace>
-      </plugin>
-    </gazebo>
     <xacro:if value="$(arg imu_enabled)">
       <gazebo>
@@ -65,5 +66,5 @@
           <updateRate>50.0</updateRate>
           <bodyName>base_link</bodyName>
-          <topicName>imu/data_compass</topicName>
+          <topicName>imu/data</topicName>
           <accelDrift>0.005 0.005 0.005</accelDrift>
           <accelGaussianNoise>0.005 0.005 0.005</accelGaussianNoise>
@@ -82,6 +83,6 @@
           <bodyName>base_link</bodyName>
           <frameId>base_link</frameId>
-          <topicName>/navsat/fix</topicName>
-          <velocityTopicName>/navsat/vel</velocityTopicName>
+          <topicName>navsat/fix</topicName>
+          <velocityTopicName>navsat/vel</velocityTopicName>
           <referenceLatitude>49.9</referenceLatitude>
           <referenceLongitude>8.9</referenceLongitude>

Commit message: Added husky description

File: husky_gazebo/urdf/description.gazebo.xacro (robot description, xacro)
@@ -3,5 +3,5 @@
 Software License Agreement (BSD)
 \file      description.gazebo.xacro
-\authors   Paul Bovbel <pbovbel@clearpathrobotics.com
+\authors   Paul Bovbel <pbovbel@clearpathrobotics.com, Devon Ash <dash@clearpathrobotics.com>
 \copyright Copyright (c) 2015, Clearpath Robotics, Inc., All rights reserved.
 Redistribution and use in source and binary forms, with or without modification, are permitted provided that

File: husky_gazebo/urdf/husky.gazebo.xacro (robot description, xacro)
@@ -3,5 +3,5 @@
 Software License Agreement (BSD)
 \file      husky.gazebo.xacro
-\authors   Paul Bovbel <pbovbel@clearpathrobotics.com
+\authors   Paul Bovbel <pbovbel@clearpathrobotics.com, Devon Ash <dash@clearpathrobotics.com>
 \copyright Copyright (c) 2015, Clearpath Robotics, Inc., All rights reserved.
 Redistribution and use in source and binary forms, with or without modification, are permitted provided that
@@ -26,4 +26,5 @@
   <xacro:arg name="gps_enabled" default="true" />
   <xacro:arg name="ur5_enabled" default="false" />
+  <xacro:arg name="kinect_enabled" default="false" />
   <xacro:include filename="$(find husky_description)/urdf/husky.urdf.xacro" />
   <xacro:include filename="$(find husky_gazebo)/urdf/sick_lms100.urdf.xacro" />
@@ -98,3 +99,20 @@
       <xacro:include filename="$(find husky_gazebo)/urdf/ur5_arm.gazebo.xacro"/>
   </xacro:if>
+  <xacro:if value="$(arg kinect_enabled)">
+      <!-- Spawn the sensor arch and attach it to the model -->
+      <xacro:include filename="$(find husky_description)/urdf/510_mm_sensor_arch.urdf.xacro"/>
+      <xacro:sensor_arch_510mm prefix="" parent="top_plate_link">
+          <origin xyz="0 0 0" rpy="0 0 0"/>
+      </xacro:sensor_arch_510mm>
+      <!-- Create kinect reference frame -->
+      <link name="kinect_frame"/>
+      <!-- Attach frame to sensor arch mount point -->
+      <joint name="kinect_frame_joint" type="fixed">
+          <origin xyz="0 0 0" rpy="0 0 0"/>
+          <parent link="sensor_arch_510mm_link"/>
+          <child link="kinect_frame"/>
+      </joint>
+      <!-- Spawn the kinect and attach it to the sensor arch -->
+      <xacro:kinect_camera_gazebo_v0 name="kinect"/>
+  </xacro:if>
 </robot>

Commit message: Pretty big refactor

File: husky_gazebo/urdf/description.gazebo.xacro (robot description, xacro)
@@ -21,6 +21,17 @@
 ARISING IN ANY WAY OUT OF THE USE OF THIS SOFTWARE, EVEN IF ADVISED OF THE POSSIBILITY OF SUCH DAMAGE.
 -->
-<robot name="husky_description" xmlns:xacro="http://ros.org/wiki/xacro">
+<robot name="husky_robot_gazebo" xmlns:xacro="http://ros.org/wiki/xacro">
+  <xacro:arg name="laser_enabled" default="true" />
+  <xacro:arg name="ur5_enabled" default="false" />
+  <xacro:arg name="kinect_enabled" default="false" />
+  <xacro:include filename="$(find husky_description)/urdf/husky.urdf.xacro" />
   <xacro:include filename="$(find husky_gazebo)/urdf/husky.gazebo.xacro" />
-  <xacro:husky_gazebo_robot />
+  <!-- Gazebo plugin for ROS Control -->
+  <gazebo>
+    <plugin name="gazebo_ros_control" filename="libgazebo_ros_control.so">
+      <robotNamespace>/</robotNamespace>
+    </plugin>
+  </gazebo>
+  <xacro:husky_robot />
+  <xacro:husky_robot_gazebo />
 </robot>

File: husky_gazebo/urdf/husky.gazebo.xacro (robot description, xacro)
@@ -21,95 +21,72 @@
 ARISING IN ANY WAY OUT OF THE USE OF THIS SOFTWARE, EVEN IF ADVISED OF THE POSSIBILITY OF SUCH DAMAGE.
 -->
-<robot name="husky_gazebo" xmlns:xacro="http://ros.org/wiki/xacro">
-  <xacro:arg name="front_laser" default="true" />
-  <xacro:arg name="imu_enabled" default="true" />
-  <xacro:arg name="gps_enabled" default="true" />
-  <xacro:arg name="ur5_enabled" default="false" />
-  <xacro:arg name="kinect_enabled" default="false" />
-  <xacro:include filename="$(find husky_description)/urdf/husky.urdf.xacro" />
-  <xacro:include filename="$(find husky_gazebo)/urdf/sick_lms100.urdf.xacro" />
-  <xacro:macro name="husky_gazebo_robot">
-    <xacro:husky_robot />
-    <!-- Gazebo plugin for ROS Control -->
+<robot name="husky_robot_gazebo" xmlns:xacro="http://ros.org/wiki/xacro">
+  <xacro:include filename="$(find husky_gazebo)/urdf/accessories/sick_lms100.gazebo.xacro"/>
+  <xacro:include filename="$(find husky_gazebo)/urdf/accessories/kinect_camera.gazebo.xacro"/>
+  <xacro:include filename="$(find ur_description)/urdf/ur5.gazebo.xacro" />
+  <xacro:macro name="husky_robot_gazebo">
     <gazebo>
-      <plugin name="gazebo_ros_control" filename="libgazebo_ros_control.so">
+      <plugin name="imu_controller" filename="libhector_gazebo_ros_imu.so">
         <robotNamespace>/</robotNamespace>
+        <updateRate>50.0</updateRate>
+        <bodyName>base_link</bodyName>
+        <topicName>imu/data</topicName>
+        <accelDrift>0.005 0.005 0.005</accelDrift>
+        <accelGaussianNoise>0.005 0.005 0.005</accelGaussianNoise>
+        <rateDrift>0.005 0.005 0.005 </rateDrift>
+        <rateGaussianNoise>0.005 0.005 0.005 </rateGaussianNoise>
+        <headingDrift>0.005</headingDrift>
+        <headingGaussianNoise>0.005</headingGaussianNoise>
       </plugin>
     </gazebo>
-    <xacro:if value="$(arg front_laser)">
-      <link name="sick_bracket_link">
-        <visual>
-          <geometry>
-            <mesh filename="package://husky_description/meshes/lidar_mount.stl" />
-          </geometry>
-          <material name="DarkGrey" />
-        </visual>
-      </link>
-      <joint name="sick_bracket" type="fixed">
-        <origin xyz="-0.12 0 0" rpy="0 0 0" />
-        <parent link="front_bumper_link" />
-        <child link="sick_bracket_link" />
-      </joint>
+    <gazebo>
+      <plugin name="gps_controller" filename="libhector_gazebo_ros_gps.so">
+        <updateRate>40</updateRate>
+        <robotNamespace>/</robotNamespace>
+        <bodyName>base_link</bodyName>
+        <frameId>base_link</frameId>
+        <topicName>navsat/fix</topicName>
+        <velocityTopicName>navsat/vel</velocityTopicName>
+        <referenceLatitude>49.9</referenceLatitude>
+        <referenceLongitude>8.9</referenceLongitude>
+        <referenceHeading>0</referenceHeading>
+        <referenceAltitude>0</referenceAltitude>
+        <drift>0.0001 0.0001 0.0001</drift>
+      </plugin>
+    </gazebo>
+    <xacro:if value="$(arg laser_enabled)">
       <gazebo reference="sick_bracket_link">
         <material>Gazebo/DarkGrey</material>
       </gazebo>
-      <xacro:sick_lms100 prefix="front" />
-      <joint name="front_laser_joint" type="fixed">
-        <origin xyz="0.07 0 0.17" rpy="0 0 0" />
-        <parent link="sick_bracket_link" />
-        <child link="front_laser" />
-      </joint>
+      <xacro:sick_lms100_gazebo prefix="base"/>
     </xacro:if>
-    <xacro:if value="$(arg imu_enabled)">
-      <gazebo>
-        <plugin name="imu_controller" filename="libhector_gazebo_ros_imu.so">
-          <robotNamespace>/</robotNamespace>
-          <updateRate>50.0</updateRate>
-          <bodyName>base_link</bodyName>
-          <topicName>imu/data</topicName>
-          <accelDrift>0.005 0.005 0.005</accelDrift>
-          <accelGaussianNoise>0.005 0.005 0.005</accelGaussianNoise>
-          <rateDrift>0.005 0.005 0.005 </rateDrift>
-          <rateGaussianNoise>0.005 0.005 0.005 </rateGaussianNoise>
-          <headingDrift>0.005</headingDrift>
-          <headingGaussianNoise>0.005</headingGaussianNoise>
-        </plugin>
+    <xacro:if value="$(arg ur5_enabled)">
+      <xacro:ur5_arm_gazebo />
+      <!--TODO, determine if should be pulled to ur5_arm_gazebo -->
+      <gazebo reference="ur5_arm_shoulder_link">
+        <selfCollide>true</selfCollide>
+      </gazebo>
+      <gazebo reference="ur5_arm_upper_arm_link">
+        <selfCollide>true</selfCollide>
+      </gazebo>
+      <gazebo reference="ur5_arm_forearm_link">
+        <selfCollide>true</selfCollide>
+      </gazebo>
+      <gazebo reference="ur5_arm_wrist_1_link">
+        <selfCollide>true</selfCollide>
+      </gazebo>
+      <gazebo reference="ur5_arm_wrist_3_link">
+       <selfCollide>true</selfCollide>
+      </gazebo>
+      <gazebo reference="ur5_arm_wrist_2_link">
+        <selfCollide>true</selfCollide>
+      </gazebo>
+      <gazebo reference="ur5_arm_ee_link">
+        <selfCollide>true</selfCollide>
       </gazebo>
     </xacro:if>
-    <xacro:if value="$(arg gps_enabled)">
-      <gazebo>
-        <plugin name="gps_controller" filename="libhector_gazebo_ros_gps.so">
-          <updateRate>40</updateRate>
-          <robotNamespace>/</robotNamespace>
-          <bodyName>base_link</bodyName>
-          <frameId>base_link</frameId>
-          <topicName>navsat/fix</topicName>
-          <velocityTopicName>navsat/vel</velocityTopicName>
-          <referenceLatitude>49.9</referenceLatitude>
-          <referenceLongitude>8.9</referenceLongitude>
-          <referenceHeading>0</referenceHeading>
-          <referenceAltitude>0</referenceAltitude>
-          <drift>0.0001 0.0001 0.0001</drift>
-        </plugin>
-      </gazebo>
+    <xacro:if value="$(arg kinect_enabled)">
+      <xacro:kinect_camera_gazebo prefix="camera"/>
     </xacro:if>
   </xacro:macro>
-  <xacro:if value="$(arg ur5_enabled)">
-      <xacro:include filename="$(find husky_description)/urdf/ur5_arm.urdf.xacro"/>
-      <xacro:include filename="$(find husky_gazebo)/urdf/ur5_arm.gazebo.xacro"/>
-  </xacro:if>
-  <xacro:if value="$(arg kinect_enabled)">
-      <!-- Spawn the sensor arch and attach it to the model -->
-      <xacro:include filename="$(find husky_description)/urdf/510_mm_sensor_arch.urdf.xacro"/>
-      <xacro:sensor_arch_510mm prefix="" parent="top_plate_link">
-          <origin xyz="-0.35 0 0.51" rpy="0 0 -3.14"/>
-      </xacro:sensor_arch_510mm>
-      <xacro:include filename="$(find husky_gazebo)/urdf/kinect_camera.urdf.xacro"/>
-      <!-- Attach frame to sensor arch mount point -->
-      <joint name="kinect_frame_joint" type="fixed">
-          <origin xyz="0 0 0" rpy="${3.14/8} 0 -${3.14/2}"/>
-          <parent link="sensor_arch_510mm_link"/>
-          <child link="kinect_frame"/>
-      </joint>
-  </xacro:if>
 </robot>
