Commit message: Add UR5 and Kinect simulation

File: husky_gazebo/urdf/husky.gazebo.xacro (robot description, xacro)
@@ -3,5 +3,5 @@
 Software License Agreement (BSD)
 \file      husky.gazebo.xacro
-\authors   Paul Bovbel <pbovbel@clearpathrobotics.com
+\authors   Paul Bovbel <pbovbel@clearpathrobotics.com, Devon Ash <dash@clearpathrobotics.com>
 \copyright Copyright (c) 2015, Clearpath Robotics, Inc., All rights reserved.
 Redistribution and use in source and binary forms, with or without modification, are permitted provided that
@@ -25,4 +25,6 @@
   <xacro:arg name="imu_enabled" default="true" />
   <xacro:arg name="gps_enabled" default="true" />
+  <xacro:arg name="ur5_enabled" default="false" />
+  <xacro:arg name="kinect_enabled" default="false" />
   <xacro:include filename="$(find husky_description)/urdf/husky.urdf.xacro" />
   <xacro:include filename="$(find husky_gazebo)/urdf/sick_lms100.urdf.xacro" />
@@ -93,3 +95,21 @@
     </xacro:if>
   </xacro:macro>
+  <xacro:if value="$(arg ur5_enabled)">
+      <xacro:include filename="$(find husky_description)/urdf/ur5_arm.urdf.xacro"/>
+      <xacro:include filename="$(find husky_gazebo)/urdf/ur5_arm.gazebo.xacro"/>
+  </xacro:if>
+  <xacro:if value="$(arg kinect_enabled)">
+      <!-- Spawn the sensor arch and attach it to the model -->
+      <xacro:include filename="$(find husky_description)/urdf/510_mm_sensor_arch.urdf.xacro"/>
+      <xacro:sensor_arch_510mm prefix="" parent="top_plate_link">
+          <origin xyz="-0.35 0 0.51" rpy="0 0 -3.14"/>
+      </xacro:sensor_arch_510mm>
+      <xacro:include filename="$(find husky_gazebo)/urdf/kinect_camera.urdf.xacro"/>
+      <!-- Attach frame to sensor arch mount point -->
+      <joint name="kinect_frame_joint" type="fixed">
+          <origin xyz="0 0 0" rpy="${3.14/8} 0 -${3.14/2}"/>
+          <parent link="sensor_arch_510mm_link"/>
+          <child link="kinect_frame"/>
+      </joint>
+  </xacro:if>
 </robot>

File: husky_gazebo/urdf/ur5_arm.gazebo.xacro (robot description, xacro)
@@ -2,6 +2,6 @@
 <!--
 Software License Agreement (BSD)
-\file      description.gazebo.xacro
-\authors   Paul Bovbel <pbovbel@clearpathrobotics.com, Devon Ash <dash@clearpathrobotics.com>
+\file      ur5_arm.gazebo.xacro
+\authors   Devon Ash <dash@clearpathrobotics.com
 \copyright Copyright (c) 2015, Clearpath Robotics, Inc., All rights reserved.
 Redistribution and use in source and binary forms, with or without modification, are permitted provided that
@@ -21,6 +21,29 @@
 ARISING IN ANY WAY OUT OF THE USE OF THIS SOFTWARE, EVEN IF ADVISED OF THE POSSIBILITY OF SUCH DAMAGE.
 -->
-<robot name="husky_description" xmlns:xacro="http://ros.org/wiki/xacro">
-  <xacro:include filename="$(find husky_gazebo)/urdf/husky.gazebo.xacro" />
-  <xacro:husky_gazebo_robot />
+<robot name="husky_ur5_arm_gazebo" xmlns:xacro="http://ros.org/wiki/xacro">
+  <gazebo reference="ur5_top_plate_link">
+     <material>Gazebo/DarkGrey</material>
+  </gazebo>
+ <!-- Gazebo references for self collide -->
+  <gazebo reference="ur5_arm_shoulder_link">
+      <selfCollide>true</selfCollide>
+  </gazebo>
+ <gazebo reference="ur5_arm_upper_arm_link">
+      <selfCollide>true</selfCollide>
+  </gazebo>
+ <gazebo reference="ur5_arm_forearm_link">
+      <selfCollide>true</selfCollide>
+  </gazebo>
+ <gazebo reference="ur5_arm_wrist_1_link">
+      <selfCollide>true</selfCollide>
+  </gazebo>
+ <gazebo reference="ur5_arm_wrist_3_link">
+      <selfCollide>true</selfCollide>
+  </gazebo>
+ <gazebo reference="ur5_arm_wrist_2_link">
+      <selfCollide>true</selfCollide>
+  </gazebo>
+ <gazebo reference="ur5_arm_ee_link">
+      <selfCollide>true</selfCollide>
+  </gazebo>
 </robot>

Commit message: Updated sensor arch

File: husky_gazebo/urdf/husky.gazebo.xacro (robot description, xacro)
@@ -103,5 +103,5 @@
       <xacro:include filename="$(find husky_description)/urdf/510_mm_sensor_arch.urdf.xacro"/>
       <xacro:sensor_arch_510mm prefix="" parent="top_plate_link">
-          <origin xyz="0 0 0" rpy="0 0 0"/>
+          <origin xyz="-0.35 0 0.51" rpy="0 0 3.14"/>
       </xacro:sensor_arch_510mm>
       <!-- Create kinect reference frame -->

Commit message: Added kinect

File: husky_gazebo/urdf/husky.gazebo.xacro (robot description, xacro)
@@ -105,6 +105,5 @@
           <origin xyz="-0.35 0 0.51" rpy="0 0 3.14"/>
       </xacro:sensor_arch_510mm>
-      <!-- Create kinect reference frame -->
-      <link name="kinect_frame"/>
+      <xacro:include filename="$(find husky_gazebo)/urdf/kinect_camera.urdf.xacro"/>
       <!-- Attach frame to sensor arch mount point -->
       <joint name="kinect_frame_joint" type="fixed">
@@ -113,6 +112,4 @@
           <child link="kinect_frame"/>
       </joint>
-      <!-- Spawn the kinect and attach it to the sensor arch -->
-      <xacro:kinect_camera_gazebo_v0 name="kinect"/>
   </xacro:if>
 </robot>

Commit message: Positioned kinect properly

File: husky_gazebo/urdf/husky.gazebo.xacro (robot description, xacro)
@@ -103,10 +103,10 @@
       <xacro:include filename="$(find husky_description)/urdf/510_mm_sensor_arch.urdf.xacro"/>
       <xacro:sensor_arch_510mm prefix="" parent="top_plate_link">
-          <origin xyz="-0.35 0 0.51" rpy="0 0 3.14"/>
+          <origin xyz="-0.35 0 0.51" rpy="0 0 -3.14"/>
       </xacro:sensor_arch_510mm>
       <xacro:include filename="$(find husky_gazebo)/urdf/kinect_camera.urdf.xacro"/>
       <!-- Attach frame to sensor arch mount point -->
       <joint name="kinect_frame_joint" type="fixed">
-          <origin xyz="0 0 0" rpy="0 0 0"/>
+          <origin xyz="0 0 0" rpy="${3.14/8} 0 -${3.14/2}"/>
           <parent link="sensor_arch_510mm_link"/>
           <child link="kinect_frame"/>

Commit message: Move into macro

File: husky_gazebo/urdf/husky.gazebo.xacro (robot description, xacro)
@@ -26,67 +26,67 @@
   <xacro:include filename="$(find ur_description)/urdf/ur5.gazebo.xacro" />
   <xacro:macro name="husky_robot_gazebo">
-      <gazebo>
-        <plugin name="imu_controller" filename="libhector_gazebo_ros_imu.so">
-          <robotNamespace>/</robotNamespace>
-          <updateRate>50.0</updateRate>
-          <bodyName>base_link</bodyName>
-          <topicName>imu/data</topicName>
-          <accelDrift>0.005 0.005 0.005</accelDrift>
-          <accelGaussianNoise>0.005 0.005 0.005</accelGaussianNoise>
-          <rateDrift>0.005 0.005 0.005 </rateDrift>
-          <rateGaussianNoise>0.005 0.005 0.005 </rateGaussianNoise>
-          <headingDrift>0.005</headingDrift>
-          <headingGaussianNoise>0.005</headingGaussianNoise>
-        </plugin>
+    <gazebo>
+      <plugin name="imu_controller" filename="libhector_gazebo_ros_imu.so">
+        <robotNamespace>/</robotNamespace>
+        <updateRate>50.0</updateRate>
+        <bodyName>base_link</bodyName>
+        <topicName>imu/data</topicName>
+        <accelDrift>0.005 0.005 0.005</accelDrift>
+        <accelGaussianNoise>0.005 0.005 0.005</accelGaussianNoise>
+        <rateDrift>0.005 0.005 0.005 </rateDrift>
+        <rateGaussianNoise>0.005 0.005 0.005 </rateGaussianNoise>
+        <headingDrift>0.005</headingDrift>
+        <headingGaussianNoise>0.005</headingGaussianNoise>
+      </plugin>
+    </gazebo>
+    <gazebo>
+      <plugin name="gps_controller" filename="libhector_gazebo_ros_gps.so">
+        <updateRate>40</updateRate>
+        <robotNamespace>/</robotNamespace>
+        <bodyName>base_link</bodyName>
+        <frameId>base_link</frameId>
+        <topicName>navsat/fix</topicName>
+        <velocityTopicName>navsat/vel</velocityTopicName>
+        <referenceLatitude>49.9</referenceLatitude>
+        <referenceLongitude>8.9</referenceLongitude>
+        <referenceHeading>0</referenceHeading>
+        <referenceAltitude>0</referenceAltitude>
+        <drift>0.0001 0.0001 0.0001</drift>
+      </plugin>
+    </gazebo>
+    <xacro:if value="$(arg laser_enabled)">
+      <gazebo reference="sick_bracket_link">
+        <material>Gazebo/DarkGrey</material>
       </gazebo>
-      <gazebo>
-        <plugin name="gps_controller" filename="libhector_gazebo_ros_gps.so">
-          <updateRate>40</updateRate>
-          <robotNamespace>/</robotNamespace>
-          <bodyName>base_link</bodyName>
-          <frameId>base_link</frameId>
-          <topicName>navsat/fix</topicName>
-          <velocityTopicName>navsat/vel</velocityTopicName>
-          <referenceLatitude>49.9</referenceLatitude>
-          <referenceLongitude>8.9</referenceLongitude>
-          <referenceHeading>0</referenceHeading>
-          <referenceAltitude>0</referenceAltitude>
-          <drift>0.0001 0.0001 0.0001</drift>
-        </plugin>
+      <xacro:sick_lms100_gazebo prefix="base"/>
+    </xacro:if>
+    <xacro:if value="$(arg ur5_enabled)">
+      <xacro:ur5_arm_gazebo />
+      <!--TODO, determine if should be pulled to ur5_arm_gazebo -->
+      <gazebo reference="ur5_arm_shoulder_link">
+        <selfCollide>true</selfCollide>
       </gazebo>
+      <gazebo reference="ur5_arm_upper_arm_link">
+        <selfCollide>true</selfCollide>
+      </gazebo>
+      <gazebo reference="ur5_arm_forearm_link">
+        <selfCollide>true</selfCollide>
+      </gazebo>
+      <gazebo reference="ur5_arm_wrist_1_link">
+        <selfCollide>true</selfCollide>
+      </gazebo>
+      <gazebo reference="ur5_arm_wrist_3_link">
+       <selfCollide>true</selfCollide>
+      </gazebo>
+      <gazebo reference="ur5_arm_wrist_2_link">
+        <selfCollide>true</selfCollide>
+      </gazebo>
+      <gazebo reference="ur5_arm_ee_link">
+        <selfCollide>true</selfCollide>
+      </gazebo>
+    </xacro:if>
+    <xacro:if value="$(arg kinect_enabled)">
+      <xacro:kinect_camera_gazebo prefix="camera"/>
+    </xacro:if>
   </xacro:macro>
-  <xacro:if value="$(arg laser_enabled)">
-    <gazebo reference="sick_bracket_link">
-      <material>Gazebo/DarkGrey</material>
-    </gazebo>
-    <xacro:sick_lms100_gazebo prefix="base"/>
-  </xacro:if>
-  <xacro:if value="$(arg ur5_enabled)">
-    <xacro:ur5_arm_gazebo />
-    <!--TODO, determine if should be pulled to ur5_arm_gazebo -->
-    <gazebo reference="ur5_arm_shoulder_link">
-      <selfCollide>true</selfCollide>
-    </gazebo>
-    <gazebo reference="ur5_arm_upper_arm_link">
-      <selfCollide>true</selfCollide>
-    </gazebo>
-    <gazebo reference="ur5_arm_forearm_link">
-      <selfCollide>true</selfCollide>
-    </gazebo>
-    <gazebo reference="ur5_arm_wrist_1_link">
-      <selfCollide>true</selfCollide>
-    </gazebo>
-    <gazebo reference="ur5_arm_wrist_3_link">
-     <selfCollide>true</selfCollide>
-    </gazebo>
-    <gazebo reference="ur5_arm_wrist_2_link">
-      <selfCollide>true</selfCollide>
-    </gazebo>
-    <gazebo reference="ur5_arm_ee_link">
-      <selfCollide>true</selfCollide>
-    </gazebo>
-  </xacro:if>
-  <xacro:if value="$(arg kinect_enabled)">
-    <xacro:kinect_camera_gazebo prefix="camera"/>
-  </xacro:if>
 </robot>

Commit message: Removed duplicate SICK laser plugin in husky_gazebo, since husky_description already contains a SICK laser plugin from the lms package.

File: husky_gazebo/urdf/husky.gazebo.xacro (robot description, xacro)
@@ -22,5 +22,4 @@
 -->
 <robot name="husky_robot_gazebo" xmlns:xacro="http://ros.org/wiki/xacro">
-  <xacro:include filename="$(find husky_gazebo)/urdf/accessories/sick_lms100.gazebo.xacro"/>
   <xacro:include filename="$(find husky_gazebo)/urdf/accessories/kinect_camera.gazebo.xacro"/>
   <xacro:macro name="husky_robot_gazebo">
@@ -54,10 +53,4 @@
       </plugin>
     </gazebo>
-    <xacro:if value="$(arg laser_enabled)">
-      <gazebo reference="sick_bracket_link">
-        <material>Gazebo/DarkGrey</material>
-      </gazebo>
-      <xacro:sick_lms100_gazebo prefix="base"/>
-    </xacro:if>
     <xacro:if value="$(arg ur5_enabled)">
       <!--Remove when https://github.com/ros-industrial/universal_robot/pull/168 is resolved -->

Commit message: Added grippers and fingertip coloring

File: husky_gazebo/urdf/husky.gazebo.xacro (robot description, xacro)
@@ -77,4 +77,84 @@
       </gazebo>
     </xacro:if>
+    <xacro:if value="$(arg robotiq_grippers_enabled)">
+        <gazebo reference="l_palm">
+            <material>Gazebo/Black</material>
+        </gazebo>
+        <gazebo reference="r_palm">
+            <material>Gazebo/Black</material>
+        </gazebo>
+ <gazebo reference="l_finger_1_link_0">
+            <material>Gazebo/Black</material>
+        </gazebo>
+<gazebo reference="r_finger_1_link_0">
+            <material>Gazebo/Black</material>
+        </gazebo>
+<gazebo reference="l_finger_1_link_1">
+            <material>Gazebo/Black</material>
+        </gazebo>
+<gazebo reference="r_finger_1_link_1">
+            <material>Gazebo/Black</material>
+        </gazebo>
+<gazebo reference="l_finger_1_link_2">
+            <material>Gazebo/Black</material>
+        </gazebo>
+<gazebo reference="r_finger_1_link_2">
+            <material>Gazebo/Black</material>
+        </gazebo>
+<gazebo reference="l_finger_1_link_3">
+            <material>Gazebo/Grey</material>
+        </gazebo>
+<gazebo reference="r_finger_1_link_3">
+            <material>Gazebo/Grey</material>
+        </gazebo>
+<gazebo reference="l_finger_2_link_0">
+            <material>Gazebo/Black</material>
+        </gazebo>
+<gazebo reference="r_finger_2_link_0">
+            <material>Gazebo/Black</material>
+        </gazebo>
+<gazebo reference="l_finger_2_link_1">
+            <material>Gazebo/Black</material>
+        </gazebo>
+<gazebo reference="r_finger_2_link_1">
+            <material>Gazebo/Black</material>
+        </gazebo>
+<gazebo reference="l_finger_2_link_2">
+            <material>Gazebo/Black</material>
+        </gazebo>
+<gazebo reference="r_finger_2_link_2">
+            <material>Gazebo/Black</material>
+        </gazebo>
+<gazebo reference="l_finger_2_link_3">
+            <material>Gazebo/Grey</material>
+        </gazebo>
+<gazebo reference="r_finger_2_link_3">
+            <material>Gazebo/Grey</material>
+        </gazebo>
+<gazebo reference="l_finger_middle_link_0">
+            <material>Gazebo/Black</material>
+        </gazebo>
+<gazebo reference="r_finger_middle_link_0">
+            <material>Gazebo/Black</material>
+        </gazebo>
+<gazebo reference="l_finger_middle_link_1">
+            <material>Gazebo/Black</material>
+        </gazebo>
+<gazebo reference="r_finger_middle_link_1">
+            <material>Gazebo/Black</material>
+        </gazebo>
+<gazebo reference="l_finger_middle_link_2">
+            <material>Gazebo/Black</material>
+        </gazebo>
+<gazebo reference="r_finger_middle_link_2">
+            <material>Gazebo/Black</material>
+        </gazebo>
+<gazebo reference="l_finger_middle_link_3">
+            <material>Gazebo/Grey</material>
+        </gazebo>
+<gazebo reference="r_finger_middle_link_3">
+            <material>Gazebo/Grey</material>
+        </gazebo>
+    </xacro:if>
     <xacro:if value="$(arg kinect_enabled)">
       <xacro:kinect_camera_gazebo prefix="camera"/>
