Commit message: Pretty big refactor

File: husky_gazebo/urdf/accessories/sick_lms100.gazebo.xacro (robot description, xacro)
@@ -28,23 +28,39 @@
   xmlns:controller="http://playerstage.sourceforge.net/gazebo/xmlschema/#controller"
   xmlns:interface="http://playerstage.sourceforge.net/gazebo/xmlschema/#interface"
-  xmlns:xacro="http://ros.org/wiki/xacro" name="kinect_camera">
-  <!-- Bring in the Gazebo plugin -->
-  <xacro:include filename="$(find husky_gazebo)/urdf/kinect_camera.gazebo.xacro"/>
-  <!-- Create kinect reference frame -->
-  <!-- Add mesh for kinect -->
-  <link name="kinect_frame">
-      <origin xyz="0 0 0" rpy="0 0 0"/>
-      <visual>
-          <geometry>
-               <mesh filename="package://husky_gazebo/meshes/kinect.dae" />
-          </geometry>
-      </visual>
-      <collision>
-          <geometry>
-               <mesh filename="package://husky_gazebo/meshes/kinect.dae" />
-          </geometry>
-      </collision>
-  </link>
-  <!-- Spawn the kinect -->
-  <xacro:kinect_camera_gazebo_v0 name="kinect"/>
+  xmlns:xacro="http://ros.org/wiki/xacro" name="sick_lms100">
+  <xacro:macro name="sick_lms100_gazebo" params="prefix">
+    <gazebo reference="${prefix}_laser">
+      <material>Gazebo/Grey</material>
+      <turnGravityOff>true</turnGravityOff>
+      <sensor type="ray" name="${prefix}_laser">
+        <pose>0 0 0 0 0 0</pose>
+        <visualize>false</visualize>
+        <update_rate>40</update_rate>
+        <ray>
+          <scan>
+            <horizontal>
+              <samples>720</samples>
+              <resolution>1</resolution>
+              <min_angle>-1.570796</min_angle>
+              <max_angle>1.570796</max_angle>
+            </horizontal>
+          </scan>
+          <range>
+            <min>0.10</min>
+            <max>6.0</max>
+            <resolution>0.01</resolution>
+          </range>
+          <noise>
+            <type>gaussian</type>
+            <mean>0.0</mean>
+            <stddev>0.001</stddev>
+          </noise>
+        </ray>
+        <plugin name="gazebo_ros_laser" filename="libgazebo_ros_laser.so">
+          <topicName>scan</topicName>
+          <frameName>${prefix}_laser</frameName>
+        </plugin>
+      </sensor>
+    </gazebo>
+  </xacro:macro>
 </robot>

File: husky_gazebo/urdf/description.gazebo.xacro (robot description, xacro)
@@ -21,5 +21,10 @@
 ARISING IN ANY WAY OUT OF THE USE OF THIS SOFTWARE, EVEN IF ADVISED OF THE POSSIBILITY OF SUCH DAMAGE.
 -->
-<robot name="husky_description" xmlns:xacro="http://ros.org/wiki/xacro">
+<robot name="husky_robot_gazebo" xmlns:xacro="http://ros.org/wiki/xacro">
+  <xacro:arg name="laser_enabled" default="true" />
+  <xacro:arg name="ur5_enabled" default="false" />
+  <xacro:arg name="kinect_enabled" default="false" />
+  <xacro:include filename="$(find husky_description)/urdf/husky.urdf.xacro" />
+  <xacro:include filename="$(find husky_gazebo)/urdf/husky.gazebo.xacro" />
   <!-- Gazebo plugin for ROS Control -->
   <gazebo>
@@ -28,5 +33,5 @@
     </plugin>
   </gazebo>
-  <xacro:include filename="$(find husky_gazebo)/urdf/husky.gazebo.xacro" />
-  <xacro:husky_gazebo_robot />
+  <xacro:husky_robot />
+  <xacro:husky_robot_gazebo />
 </robot>

File: husky_gazebo/urdf/husky.gazebo.xacro (robot description, xacro)
@@ -21,39 +21,9 @@
 ARISING IN ANY WAY OUT OF THE USE OF THIS SOFTWARE, EVEN IF ADVISED OF THE POSSIBILITY OF SUCH DAMAGE.
 -->
-<robot name="husky_gazebo" xmlns:xacro="http://ros.org/wiki/xacro">
-  <xacro:arg name="front_laser" default="true" />
-  <xacro:arg name="imu_enabled" default="true" />
-  <xacro:arg name="gps_enabled" default="true" />
-  <xacro:arg name="ur5_enabled" default="false" />
-  <xacro:arg name="kinect_enabled" default="false" />
-  <xacro:include filename="$(find husky_description)/urdf/husky.urdf.xacro" />
-  <xacro:include filename="$(find husky_gazebo)/urdf/sick_lms100.urdf.xacro" />
-  <xacro:macro name="husky_gazebo_robot">
-    <xacro:husky_robot />
-    <xacro:if value="$(arg front_laser)">
-      <link name="sick_bracket_link">
-        <visual>
-          <geometry>
-            <mesh filename="package://husky_description/meshes/lidar_mount.stl" />
-          </geometry>
-          <material name="DarkGrey" />
-        </visual>
-      </link>
-      <joint name="sick_bracket" type="fixed">
-        <origin xyz="-0.12 0 0" rpy="0 0 0" />
-        <parent link="front_bumper_link" />
-        <child link="sick_bracket_link" />
-      </joint>
-      <gazebo reference="sick_bracket_link">
-        <material>Gazebo/DarkGrey</material>
-      </gazebo>
-      <xacro:sick_lms100 prefix="front" />
-      <joint name="front_laser_joint" type="fixed">
-        <origin xyz="0.07 0 0.17" rpy="0 0 0" />
-        <parent link="sick_bracket_link" />
-        <child link="front_laser" />
-      </joint>
-    </xacro:if>
-    <xacro:if value="$(arg imu_enabled)">
+<robot name="husky_robot_gazebo" xmlns:xacro="http://ros.org/wiki/xacro">
+  <xacro:include filename="$(find husky_gazebo)/urdf/accessories/sick_lms100.gazebo.xacro"/>
+  <xacro:include filename="$(find husky_gazebo)/urdf/accessories/kinect_camera.gazebo.xacro"/>
+  <xacro:include filename="$(find ur_description)/urdf/ur5.gazebo.xacro" />
+  <xacro:macro name="husky_robot_gazebo">
       <gazebo>
         <plugin name="imu_controller" filename="libhector_gazebo_ros_imu.so">
@@ -70,6 +40,4 @@
         </plugin>
       </gazebo>
-    </xacro:if>
-    <xacro:if value="$(arg gps_enabled)">
       <gazebo>
         <plugin name="gps_controller" filename="libhector_gazebo_ros_gps.so">
@@ -87,23 +55,38 @@
         </plugin>
       </gazebo>
-    </xacro:if>
   </xacro:macro>
+  <xacro:if value="$(arg laser_enabled)">
+    <gazebo reference="sick_bracket_link">
+      <material>Gazebo/DarkGrey</material>
+    </gazebo>
+    <xacro:sick_lms100_gazebo prefix="base"/>
+  </xacro:if>
   <xacro:if value="$(arg ur5_enabled)">
-      <xacro:include filename="$(find husky_description)/urdf/ur5_arm.urdf.xacro"/>
-      <xacro:include filename="$(find husky_gazebo)/urdf/ur5_arm.gazebo.xacro"/>
+    <xacro:ur5_arm_gazebo />
+    <!--TODO, determine if should be pulled to ur5_arm_gazebo -->
+    <gazebo reference="ur5_arm_shoulder_link">
+      <selfCollide>true</selfCollide>
+    </gazebo>
+    <gazebo reference="ur5_arm_upper_arm_link">
+      <selfCollide>true</selfCollide>
+    </gazebo>
+    <gazebo reference="ur5_arm_forearm_link">
+      <selfCollide>true</selfCollide>
+    </gazebo>
+    <gazebo reference="ur5_arm_wrist_1_link">
+      <selfCollide>true</selfCollide>
+    </gazebo>
+    <gazebo reference="ur5_arm_wrist_3_link">
+     <selfCollide>true</selfCollide>
+    </gazebo>
+    <gazebo reference="ur5_arm_wrist_2_link">
+      <selfCollide>true</selfCollide>
+    </gazebo>
+    <gazebo reference="ur5_arm_ee_link">
+      <selfCollide>true</selfCollide>
+    </gazebo>
   </xacro:if>
   <xacro:if value="$(arg kinect_enabled)">
-      <!-- Spawn the sensor arch and attach it to the model -->
-      <xacro:include filename="$(find husky_description)/urdf/510_mm_sensor_arch.urdf.xacro"/>
-      <xacro:sensor_arch_510mm prefix="" parent="top_plate_link">
-          <origin xyz="-0.35 0 0.51" rpy="0 0 -3.14"/>
-      </xacro:sensor_arch_510mm>
-      <xacro:include filename="$(find husky_gazebo)/urdf/kinect_camera.urdf.xacro"/>
-      <!-- Attach frame to sensor arch mount point -->
-      <joint name="kinect_frame_joint" type="fixed">
-          <origin xyz="0 0 0" rpy="${3.14/8} 0 -${3.14/2}"/>
-          <parent link="sensor_arch_510mm_link"/>
-          <child link="kinect_frame"/>
-      </joint>
+    <xacro:kinect_camera_gazebo prefix="camera"/>
   </xacro:if>
 </robot>
