Commit message: Correct frame naming convention

File: husky_gazebo/urdf/accessories/kinect_camera.gazebo.xacro (robot description, xacro)
@@ -5,7 +5,7 @@
     <origin xyz="0 0 0" rpy="-1.5708 0 -1.5708"/>
     <parent link="${prefix}_link"/>
-    <child link="${prefix}_optical_frame"/>
+    <child link="${prefix}_frame_optical"/>
   </joint>
-  <link name="${prefix}_optical_frame"/>
+  <link name="${prefix}_frame_optical"/>
   <gazebo reference="${prefix}_link">
     <sensor type="depth" name="${prefix}">
@@ -33,5 +33,5 @@
         <cameraInfoTopicName>rgb/camera_info</cameraInfoTopicName>
         <depthImageCameraInfoTopicName>depth/camera_info</depthImageCameraInfoTopicName>
-        <frameName>${prefix}_optical_frame</frameName>
+        <frameName>${prefix}_frame_optical</frameName>
         <baseline>0.1</baseline>
         <distortion_k1>0.0</distortion_k1>
